File: Schematics/ECE5 v2.kicad_pcb (KiCad board)
At the start: 2 copper layers, 150 x 100 mm, 74 parts, among them J1 AudioJack3_SwitchTR, J2 AudioJack3_SwitchTR, J3 Conn_02x08_Odd_Even, J4 Conn_02x08_Odd_Even, J5 Barrel_Jack_MountingPin, J6 Conn_02x08_Odd_Even, J7 Conn_01x02_Female, Q1 2N3904, Q2 2N3904, Q3 2N3904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

Commit message: Finalized PCB
Parts:
- moved A1 117.6 mm to (150.0, 100.5), turned to 270 degrees
- moved C1 62.6 mm to (36.8, 105.1), turned to 180 degrees
- moved C4 59.6 mm to (36.8, 108.1), turned to 180 degrees
- moved T2 57.4 mm to (64.3, 86.5)
- moved T1 49.5 mm to (81.4, 86.5)
- moved C2 47.8 mm to (40.0, 115.9), turned to 0 degrees
- moved U4 45.5 mm to (47.6, 112.7), turned to 180 degrees
- moved R20 42.4 mm to (39.5, 119.5), turned to 0 degrees
- moved J7 40.4 mm to (60.5, 109.4)
- moved C3 38.7 mm to (51.6, 112.5)
- moved R14 38.0 mm to (69.4, 96.7), turned to 180 degrees
- moved R13 30.4 mm to (76.4, 96.7)
- moved R19 22.1 mm to (63.7, 119.5), turned to 180 degrees
- moved R40 15.9 mm to (143.7, 45.9)
- moved R37 6.35 mm to (134.1, 56.0)
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Routing:
- net +5V: track 0.00 -> 284.7 mm, vias 0 -> 4
- net Net-(J2-PadR): track 0.00 -> 201.3 mm
- net Net-(J2-PadT): track 0.00 -> 191.7 mm, vias 0 -> 1
- net Net-(J1-PadR): track 0.00 -> 182.6 mm
- net Net-(J1-PadS): track 0.00 -> 180.6 mm
- net Net-(J1-PadT): track 0.00 -> 180.0 mm, vias 0 -> 1
- net S_CLK: track 0.00 -> 142.5 mm
- net S_LATCH: track 0.00 -> 141.9 mm
- net VOL_SENSE: track 0.00 -> 135.4 mm, vias 0 -> 1
- net EQ_RST: track 0.00 -> 88.6 mm
- net Net-(U2-Pad9): track 0.00 -> 82.9 mm
- net EQ_OUT: track 0.00 -> 80.3 mm
- net S_DATA: track 0.00 -> 78.3 mm, vias 0 -> 1
- net EQ_STROBE: track 0.00 -> 76.4 mm
- net Net-(J6-Pad5): track 0.00 -> 67.6 mm
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- added copper zone on B.Cu, net GND
Other:
- board text added: "Hunter Larson 2023"
- board text added: "JLCJLCJLCJLC"
